File: v2/kicad/sbc6526.sch (KiCad schematic (older format))
At the start: 0 parts

Commit message: new revision - dual 6526
new revision - dual 6526
Changed lines of the file:
@@
 F7 "R~W" I L 6400 2900 50
 F8 "~PHI2" I L 6400 3000 50
+F9 "~CIAEXT" O R 7700 2950 50
 $EndSheet
 Wire Bus Line
@@
 F13 "TODENABLE" O L 9150 2350 50
 F14 "VPB[4..7]" I R 10450 3400 50
+F15 "~CIAEXT" I L 9150 2950 50
 $EndSheet
 Wire Bus Line
@@
 F1 "power.sch" 50
 $EndSheet
+Wire Wire Line
+	7700 2950 9150 2950
 $EndSCHEMATC

Commit message: Changing to Dual CIA
Changed lines of the file:
@@
 Wire Wire Line
 	8850 4050 8850 3400
-$Sheet
-S 4200 6050 850  900
-U 5FB325FD
-F0 "clockmeter" 50
-F1 "clockmeter.sch" 50
-F2 "PHI2" I R 5050 6200 50
-$EndSheet
-Wire Wire Line
-	5750 4900 5750 6200
-Connection ~ 5750 4900
 Wire Bus Line
 	8900 1000 8900 2000
@@
 Wire Bus Line
 	900  1100 3400 1100
-Wire Wire Line
-	5050 6200 5750 6200
 Wire Bus Line
 	10450 3500 10900 3500
@@
 Wire Wire Line
 	7700 2950 9150 2950
+$Sheet
+S 4200 6050 850  900
+U 5FB325FD
+F0 "clockmeter" 50
+F1 "clockmeter.sch" 50
+F2 "~PHI2" I R 5050 6200 50
+$EndSheet
+Wire Wire Line
+	5050 6200 5650 6200
+Wire Wire Line
+	5650 6200 5650 5000
+Connection ~ 5650 5000
 $EndSCHEMATC
