File: v2/kicad/clockmeter.kicad_sch (KiCad schematic)
At the start: 14 parts, among them Y1 20M

Commit message: PCB Tweaks
Tracks optimized.
SMD components moved to top layer.
Changed lines of the file:
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@@
     (stroke (width 0) (type solid) (color 0 0 0 0))
+  )
+  (label "LEDBUS" (at 104.14 90.17 270)
+    (effects (font (size 1.27 1.27)) (justify right bottom))
   )
   (label "D" (at 107.95 50.8 0)
