File: kicad/clockmeter.kicad_sch (KiCad schematic)
At the start: 14 parts, among them Y1 20M

Commit message: v2.0
Production ready
Other:
- company: (none) -> Daniel Molina García
- title: (none) -> SBC6526 - ClockMeter
Changed lines of the file:
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@@
 (kicad_sch (version 20201015) (generator eeschema)
   (paper "A4")
+  (title_block
+    (title "SBC6526 - ClockMeter")
+    (date "2021-10-01")
+    (rev "2.0")
+    (company "Daniel Molina García")
+  )
   (bus_alias "LEDBUS" (members "A" "B" "C" "D" "E" "F" "G" "DP"))
   (junction (at 185.42 74.93) (diameter 1.016) (color 0 0 0 0))

Commit message: Uploaded firmware v2.0.2
Connections:
- net ~PHI2 renamed ~{PHI2}
