File: kicad/cpu.kicad_sch (KiCad schematic)
At the start: 3 parts, among them U3 W65C02SxP

Commit message: v2.0
Production ready
Other:
- company: (none) -> Daniel Molina García
- title: (none) -> SBC6526 - CPU
Changed lines of the file:
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@@
 (kicad_sch (version 20201015) (generator eeschema)
   (paper "A4")
+  (title_block
+    (title "SBC6526 - CPU")
+    (date "2021-10-01")
+    (rev "2.0")
+    (company "Daniel Molina García")
+  )
   (junction (at 71.12 93.98) (diameter 1.016) (color 0 0 0 0))
   (no_connect (at 142.24 127))
-  (no_connect (at 142.24 121.92))
   (no_connect (at 142.24 86.36))
   (no_connect (at 142.24 83.82))
+  (no_connect (at 142.24 121.92))
   (no_connect (at 142.24 124.46))
   (bus_entry (at 181.61 73.66) (size 2.54 -2.54)

Commit message: Uploaded firmware v2.0.2
Connections:
- net R~W renamed R~{W}
- net ~IRQ renamed ~{IRQ}
- net ~RES renamed ~{RES}
- net ~VIAIRQ renamed ~{VIAIRQ}
