File: kicad/io.kicad_sch (KiCad schematic)
At the start: 9 parts, among them SW1 UP, SW2 DOWN, SW3 OK, SW4 CANCEL

Commit message: v2.0
Production ready
Other:
- company: (none) -> Daniel Molina García
- title: (none) -> SBC6526 - IO
Changed lines of the file:
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@@
 (kicad_sch (version 20201015) (generator eeschema)
   (paper "A4")
+  (title_block
+    (title "SBC6526 - IO")
+    (date "2021-10-01")
+    (rev "2.0")
+    (company "Daniel Molina García")
+  )
   (junction (at 241.3 76.2) (diameter 1.016) (color 0 0 0 0))
   (junction (at 241.3 90.17) (diameter 1.016) (color 0 0 0 0))
