File: kicad/clock.kicad_sch (KiCad schematic)
At the start: 4 parts, among them P1 2k, U7 74AC74, U8 74AC14

Commit message: v2.0
Production ready
Other:
- company: (none) -> Daniel Molina García
- title: (none) -> SBC6526 - Clock Generator
Changed lines of the file:
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@@
 (kicad_sch (version 20201015) (generator eeschema)
   (paper "A4")
+  (title_block
+    (title "SBC6526 - Clock Generator")
+    (date "2021-10-01")
+    (rev "2.0")
+    (company "Daniel Molina García")
+  )
   (junction (at 93.98 100.33) (diameter 1.016) (color 0 0 0 0))
   (junction (at 124.46 88.9) (diameter 1.016) (color 0 0 0 0))

Commit message: Uploaded firmware v2.0.2
Connections:
- net ~PHI2 renamed ~{PHI2}
Changed lines of the file:
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@@
-(kicad_sch (version 20201015) (generator eeschema)
+(kicad_sch (version 20211123) (generator eeschema)
   (paper "A4")
   (title_block
@@
     (company "Daniel Molina García")
   )
-  (junction (at 93.98 100.33) (diameter 1.016) (color 0 0 0 0))
-  (junction (at 124.46 88.9) (diameter 1.016) (color 0 0 0 0))
-  (junction (at 194.31 91.44) (diameter 1.016) (color 0 0 0 0))
+  (junction (at 93.98 100.33) (diameter 1.016) (color 0 0 0 0)
+  )
+  (junction (at 124.46 88.9) (diameter 1.016) (color 0 0 0 0)
+  )
+  (junction (at 194.31 91.44) (diameter 1.016) (color 0 0 0 0)
+  )
   (no_connect (at 128.27 100.33))
-  (wire (pts (xy 93.98 88.9) (xy 93.98 100.33))
-    (stroke (width 0) (type solid) (color 0 0 0 0))
-  )
-  (wire (pts (xy 93.98 100.33) (xy 93.98 102.87))
+  (wire (pts (xy 167.64 86.36) (xy 167.64 102.87))
     (stroke (width 0) (type solid) (color 0 0 0 0))
   )
@@
     (stroke (width 0) (type solid) (color 0 0 0 0))
   )
-  (wire (pts (xy 100.33 88.9) (xy 93.98 88.9))
+  (wire (pts (xy 194.31 102.87) (xy 194.31 91.44))
     (stroke (width 0) (type solid) (color 0 0 0 0))
   )
@@
     (stroke (width 0) (type solid) (color 0 0 0 0))
   )
-  (wire (pts (xy 120.65 100.33) (xy 93.98 100.33))
+  (wire (pts (xy 124.46 88.9) (xy 134.62 88.9))
     (stroke (width 0) (type solid) (color 0 0 0 0))
   )
-  (wire (pts (xy 124.46 88.9) (xy 134.62 88.9))
+  (wire (pts (xy 93.98 88.9) (xy 93.98 100.33))
+    (stroke (width 0) (type solid) (color 0 0 0 0))
+  )
+  (wire (pts (xy 194.31 91.44) (xy 210.82 91.44))
+    (stroke (width 0) (type solid) (color 0 0 0 0))
+  )
+  (wire (pts (xy 172.72 86.36) (xy 167.64 86.36))
     (stroke (width 0) (type solid) (color 0 0 0 0))
   )
@@
     (stroke (width 0) (type solid) (color 0 0 0 0))
   )
-  (wire (pts (xy 167.64 86.36) (xy 167.64 102.87))
+  (wire (pts (xy 93.98 100.33) (xy 93.98 102.87))
     (stroke (width 0) (type solid) (color 0 0 0 0))
   )
@@
     (stroke (width 0) (type solid) (color 0 0 0 0))
   )
-  (wire (pts (xy 172.72 86.36) (xy 167.64 86.36))
+  (wire (pts (xy 187.96 91.44) (xy 194.31 91.44))
+    (stroke (width 0) (type solid) (color 0 0 0 0))
+  )
+  (wire (pts (xy 120.65 100.33) (xy 93.98 100.33))
     (stroke (width 0) (type solid) (color 0 0 0 0))
   )
@@
     (stroke (width 0) (type solid) (color 0 0 0 0))
   )
-  (wire (pts (xy 187.96 91.44) (xy 194.31 91.44))
-    (stroke (width 0) (type solid) (color 0 0 0 0))
-  )
-  (wire (pts (xy 194.31 91.44) (xy 210.82 91.44))
-    (stroke (width 0) (type solid) (color 0 0 0 0))
-  )
-  (wire (pts (xy 194.31 102.87) (xy 194.31 91.44))
+  (wire (pts (xy 100.33 88.9) (xy 93.98 88.9))
     (stroke (width 0) (type solid) (color 0 0 0 0))
   )
@@
     (effects (font (size 1.27 1.27)) (justify left))
   )
-  (hierarchical_label "~PHI2" (shape output) (at 210.82 91.44 0)
+  (hierarchical_label "~{PHI2}" (shape output) (at 210.82 91.44 0)
     (effects (font (size 1.27 1.27)) (justify left))
   )
-  (symbol (lib_id "power:VCC") (at 180.34 81.28 0) (unit 1)
+  (symbol (lib_id "74xx:74LS14") (at 107.95 88.9 0) (unit 1)
     (in_bom yes) (on_board yes)
-    (property "Reference" "#PWR0102" (id 0) (at 180.34 85.09 0)
+    (property "Reference" "U8" (id 0) (at 107.95 80.8482 0))
+    (property "Value" "74AC14" (id 1) (at 107.95 83.1596 0))
+    (property "Footprint" "Package_SO:SOIC-14_3.9x8.7mm_P1.27mm" (id 2) (at 107.95 88.9 0)
       (effects (font (size 1.27 1.27)) hide)
     )
-    (property "Value" "VCC" (id 1) (at 180.721 76.8858 0))
-    (property "Footprint" "" (id 2) (at 180.34 81.28 0)
+    (property "Datasheet" "http://www.ti.com/lit/gpn/sn74LS14" (id 3) (at 107.95 88.9 0)
       (effects (font (size 1.27 1.27)) hide)
     )
-    (property "Datasheet" "" (id 3) (at 180.34 81.28 0)
+    (pin "1")
+    (pin "2")
+  )
+  (symbol (lib_id "74xx:74LS14") (at 142.24 88.9 0) (unit 2)
+    (in_bom yes) (on_board yes)
+    (property "Reference" "U8" (id 0) (at 142.24 80.8482 0))
+    (property "Value" "74AC14" (id 1) (at 142.24 83.1596 0))
+    (property "Footprint" "Package_SO:SOIC-14_3.9x8.7mm_P1.27mm" (id 2) (at 142.24 88.9 0)
       (effects (font (size 1.27 1.27)) hide)
     )
-  )
-  (symbol (lib_id "power:VCC") (at 180.34 96.52 180) (unit 1)
-    (in_bom yes) (on_board yes)
-    (property "Reference" "#PWR0103" (id 0) (at 180.34 92.71 0)
+    (property "Datasheet" "http://www.ti.com/lit/gpn/sn74LS14" (id 3) (at 142.24 88.9 0)
       (effects (font (size 1.27 1.27)) hide)
     )
-    (property "Value" "VCC" (id 1) (at 179.959 100.9142 0))
-    (property "Footprint" "" (id 2) (at 180.34 96.52 0)
+    (pin "3")
+    (pin "4")
+  )
+  (symbol (lib_id "74xx:74LS74") (at 180.34 88.9 0) (unit 2)
+    (in_bom yes) (on_board yes)
+    (property "Reference" "U7" (id 0) (at 185.42 77.47 0))
+    (property "Value" "74AC74" (id 1) (at 187.96 80.01 0))
+    (property "Footprint" "Package_SO:SOIC-14_3.9x8.7mm_P1.27mm" (id 2) (at 180.34 88.9 0)
       (effects (font (size 1.27 1.27)) hide)
     )
-    (property "Datasheet" "" (id 3) (at 180.34 96.52 0)
+    (property "Datasheet" "74xx/74hc_hct74.pdf" (id 3) (at 180.34 88.9 0)
       (effects (font (size 1.27 1.27)) hide)
     )
-  )
-  (symbol (lib_id "power:GND") (at 93.98 116.84 0) (unit 1)
-    (in_bom yes) (on_board yes)
-    (property "Reference" "#PWR0101" (id 0) (at 93.98 123.19 0)
-      (effects (font (size 1.27 1.27)) hide)
-    )
-    (property "Value" "GND" (id 1) (at 94.107 121.2342 0))
-    (property "Footprint" "" (id 2) (at 93.98 116.84 0)
-      (effects (font (size 1.27 1.27)) hide)
-    )
-    (property "Datasheet" "" (id 3) (at 93.98 116.84 0)
-      (effects (font (size 1.27 1.27)) hide)
-    )
+    (pin "10")
+    (pin "11")
+    (pin "12")
+    (pin "13")
+    (pin "8")
+    (pin "9")
   )
   (symbol (lib_id "Device:C") (at 93.98 106.68 0) (unit 1)
@@
       (effects (font (size 1.27 1.27)) hide)
     )
+    (pin "1")
+    (pin "2")
   )
   (symbol (lib_id "Device:R_POT_TRIM") (at 124.46 100.33 90) (unit 1)
@@
       (effects (font (size 1.27 1.27)) hide)
     )
+    (pin "1")
+    (pin "2")
+    (pin "3")
   )
-  (symbol (lib_id "74xx:74LS14") (at 107.95 88.9 0) (unit 1)
+  (symbol (lib_id "power:GND") (at 93.98 116.84 0) (unit 1)
     (in_bom yes) (on_board yes)
-    (property "Reference" "U8" (id 0) (at 107.95 80.8482 0))
-    (property "Value" "74AC14" (id 1) (at 107.95 83.1596 0))
-    (property "Footprint" "Package_SO:SOIC-14_3.9x8.7mm_P1.27mm" (id 2) (at 107.95 88.9 0)
+    (property "Reference" "#PWR0101" (id 0) (at 93.98 123.19 0)
       (effects (font (size 1.27 1.27)) hide)
     )
-    (property "Datasheet" "http://www.ti.com/lit/gpn/sn74LS14" (id 3) (at 107.95 88.9 0)
+    (property "Value" "GND" (id 1) (at 94.107 121.2342 0))
+    (property "Footprint" "" (id 2) (at 93.98 116.84 0)
       (effects (font (size 1.27 1.27)) hide)
     )
-  )
-  (symbol (lib_id "74xx:74LS14") (at 142.24 88.9 0) (unit 2)
-    (in_bom yes) (on_board yes)
-    (property "Reference" "U8" (id 0) (at 142.24 80.8482 0))
-    (property "Value" "74AC14" (id 1) (at 142.24 83.1596 0))
-    (property "Footprint" "Package_SO:SOIC-14_3.9x8.7mm_P1.27mm" (id 2) (at 142.24 88.9 0)
+    (property "Datasheet" "" (id 3) (at 93.98 116.84 0)
       (effects (font (size 1.27 1.27)) hide)
     )
-    (property "Datasheet" "http://www.ti.com/lit/gpn/sn74LS14" (id 3) (at 142.24 88.9 0)
+    (pin "1")
+  )
+  (symbol (lib_id "power:VCC") (at 180.34 81.28 0) (unit 1)
+    (in_bom yes) (on_board yes)
+    (property "Reference" "#PWR0102" (id 0) (at 180.34 85.09 0)
       (effects (font (size 1.27 1.27)) hide)
     )
-  )
-  (symbol (lib_id "74xx:74LS74") (at 180.34 88.9 0) (unit 2)
-    (in_bom yes) (on_board yes)
-    (property "Reference" "U7" (id 0) (at 185.42 77.47 0))
-    (property "Value" "74AC74" (id 1) (at 187.96 80.01 0))
-    (property "Footprint" "Package_SO:SOIC-14_3.9x8.7mm_P1.27mm" (id 2) (at 180.34 88.9 0)
+    (property "Value" "VCC" (id 1) (at 180.721 76.8858 0))
+    (property "Footprint" "" (id 2) (at 180.34 81.28 0)
       (effects (font (size 1.27 1.27)) hide)
     )
-    (property "Datasheet" "74xx/74hc_hct74.pdf" (id 3) (at 180.34 88.9 0)
+    (property "Datasheet" "" (id 3) (at 180.34 81.28 0)
       (effects (font (size 1.27 1.27)) hide)
     )
+    (pin "1")
+  )
+  (symbol (lib_id "power:VCC") (at 180.34 96.52 180) (unit 1)
+    (in_bom yes) (on_board yes)
+    (property "Reference" "#PWR0103" (id 0) (at 180.34 92.71 0)
+      (effects (font (size 1.27 1.27)) hide)
+    )
+    (property "Value" "VCC" (id 1) (at 179.959 100.9142 0))
+    (property "Footprint" "" (id 2) (at 180.34 96.52 0)
+      (effects (font (size 1.27 1.27)) hide)
+    )
+    (property "Datasheet" "" (id 3) (at 180.34 96.52 0)
+      (effects (font (size 1.27 1.27)) hide)
+    )
+    (pin "1")
   )
 )
