File: kicad/memory.kicad_sch (KiCad schematic)
At the start: 3 parts, among them U10 74AC138, U4 IS61C1024AL-12KLI, U9 74AC139

Commit message: v2.0
Production ready
Other:
- company: (none) -> Daniel Molina García
- title: (none) -> SBC6526 - Memory
Changed lines of the file:
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@@
 (kicad_sch (version 20201015) (generator eeschema)
   (paper "A4")
+  (title_block
+    (title "SBC6526 - Memory")
+    (date "2021-10-01")
+    (rev "2.0")
+    (company "Daniel Molina García")
+  )
   (junction (at 139.7 162.56) (diameter 1.016) (color 0 0 0 0))
-  (no_connect (at 167.64 165.1))
-  (no_connect (at 167.64 157.48))
+  (no_connect (at 167.64 160.02))
+  (no_connect (at 167.64 60.96))
+  (no_connect (at 167.64 105.41))
   (no_connect (at 167.64 128.27))
-  (no_connect (at 167.64 147.32))
-  (no_connect (at 167.64 105.41))
-  (no_connect (at 167.64 107.95))
-  (no_connect (at 167.64 162.56))
-  (no_connect (at 167.64 60.96))
-  (no_connect (at 167.64 160.02))
   (no_connect (at 167.64 113.03))
   (no_connect (at 167.64 123.19))
+  (no_connect (at 167.64 165.1))
+  (no_connect (at 167.64 162.56))
+  (no_connect (at 167.64 147.32))
+  (no_connect (at 167.64 107.95))
+  (no_connect (at 167.64 157.48))
   (bus_entry (at 134.62 38.1) (size -2.54 -2.54)
     (stroke (width 0.1524) (type solid) (color 0 0 0 0))

Commit message: Fixed Freq. Meter footprint
Frequency meter footprint was wrong. Top row was reversed.

Minor additions to bootstrap and firmware.
Other:
- note added: "11xx xxxx xxxx xxxx RAM C000 - ffff 1001 1xxx xxxx xxxx CIAEXT 9800 - 9fff 1001 0xxx xxxx xxxx VIA 9000 - 97ff 1000 1xxx xxxx xxxx CIA 8800 - 8fff 0xxx xxxx xxxx xxxx RAM 0000 - 7fff"
- note removed: "11xx xxxx xxxx xxxx RAM C000 - ffff 1001 0xxx xxxx xxxx VIA 9000 - 97ff 1000 1xxx xxxx xxxx CIA 8800 - 8fff 0xxx xxxx xxxx xxxx RAM 0000 - 7fff"
Changed lines of the file:
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@@
   )
   (junction (at 139.7 162.56) (diameter 1.016) (color 0 0 0 0))
-  (no_connect (at 167.64 160.02))
-  (no_connect (at 167.64 60.96))
   (no_connect (at 167.64 105.41))
   (no_connect (at 167.64 128.27))
+  (no_connect (at 167.64 107.95))
   (no_connect (at 167.64 113.03))
+  (no_connect (at 167.64 162.56))
+  (no_connect (at 167.64 157.48))
+  (no_connect (at 167.64 60.96))
+  (no_connect (at 167.64 165.1))
+  (no_connect (at 167.64 160.02))
   (no_connect (at 167.64 123.19))
-  (no_connect (at 167.64 165.1))
-  (no_connect (at 167.64 162.56))
   (no_connect (at 167.64 147.32))
-  (no_connect (at 167.64 107.95))
-  (no_connect (at 167.64 157.48))
   (bus_entry (at 134.62 38.1) (size -2.54 -2.54)
     (stroke (width 0.1524) (type solid) (color 0 0 0 0))
@@
     (stroke (width 0) (type solid) (color 0 0 0 0))
   )
-  (text "11xx xxxx xxxx xxxx      RAM    C000 - ffff\n1001 0xxx xxxx xxxx     VIA     9000 - 97ff\n1000 1xxx xxxx xxxx     CIA      8800 - 8fff\n0xxx xxxx xxxx xxxx      RAM     0000 - 7fff"
+  (text "11xx xxxx xxxx xxxx      RAM    C000 - ffff\n1001 1xxx xxxx xxxx    CIAEXT 9800 - 9fff\n1001 0xxx xxxx xxxx     VIA     9000 - 97ff\n1000 1xxx xxxx xxxx     CIA      8800 - 8fff\n0xxx xxxx xxxx xxxx      RAM     0000 - 7fff\n"
     (at 48.26 50.8 0)
-    (effects (font (size 1.27 1.27)) (justify left bottom))
+    (effects (font (size 1.27 1.27) (thickness 0.254) bold) (justify left bottom))
   )
   (label "A11" (at 135.89 147.32 0)

Commit message: Fixes
* Minor fixes to routing
* Right VCC hole was slightly offset. Fixed
* Removed /CE from arduino to RAM. As RAMCE pulses with PHI, it's not necessary, and we leave /CE tied to GND.
* Fixed RAM footprint, as it was too wide. Improved routing.
* Added current limiting resistor to LCD Contrast
Connections:
- net ~CE is gone; now on net GND: U4.22 (~CE1~)
- net A11: now also U4.31 (A15); no longer U4.3 (A14)
- net A12: now also U4.3 (A14); no longer U4.31 (A15)
Changed lines of the file:
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@@
   )
   (junction (at 139.7 162.56) (diameter 1.016) (color 0 0 0 0))
+  (junction (at 170.18 83.82) (diameter 1.016) (color 0 0 0 0))
+  (no_connect (at 167.64 113.03))
+  (no_connect (at 167.64 60.96))
   (no_connect (at 167.64 105.41))
+  (no_connect (at 167.64 147.32))
+  (no_connect (at 167.64 107.95))
+  (no_connect (at 167.64 165.1))
+  (no_connect (at 167.64 157.48))
+  (no_connect (at 167.64 123.19))
   (no_connect (at 167.64 128.27))
-  (no_connect (at 167.64 107.95))
-  (no_connect (at 167.64 113.03))
   (no_connect (at 167.64 162.56))
-  (no_connect (at 167.64 157.48))
-  (no_connect (at 167.64 60.96))
-  (no_connect (at 167.64 165.1))
   (no_connect (at 167.64 160.02))
-  (no_connect (at 167.64 123.19))
-  (no_connect (at 167.64 147.32))
   (bus_entry (at 134.62 38.1) (size -2.54 -2.54)
     (stroke (width 0.1524) (type solid) (color 0 0 0 0))
@@
     (stroke (width 0) (type solid) (color 0 0 0 0))
   )
-  (wire (pts (xy 167.64 71.12) (xy 233.68 71.12))
+  (wire (pts (xy 167.64 71.12) (xy 170.18 71.12))
     (stroke (width 0) (type solid) (color 0 0 0 0))
   )
@@
   )
   (wire (pts (xy 167.64 154.94) (xy 229.87 154.94))
+    (stroke (width 0) (type solid) (color 0 0 0 0))
+  )
+  (wire (pts (xy 170.18 71.12) (xy 170.18 83.82))
     (stroke (width 0) (type solid) (color 0 0 0 0))
   )
@@
     (effects (font (size 1.27 1.27)) (justify left bottom))
   )
-  (label "A11" (at 137.16 73.66 0)
-    (effects (font (size 1.27 1.27)) (justify left bottom))
-  )
-  (label "A12" (at 137.16 76.2 0)
+  (label "A12" (at 137.16 73.66 0)
+    (effects (font (size 1.27 1.27)) (justify left bottom))
+  )
+  (label "A11" (at 137.16 76.2 0)
     (effects (font (size 1.27 1.27)) (justify left bottom))
   )
@@
   )
   (label "~CIAEXT" (at 170.18 154.94 0)
-    (effects (font (size 1.27 1.27)) (justify left bottom))
-  )
-  (label "~CE" (at 175.26 71.12 0)
     (effects (font (size 1.27 1.27)) (justify left bottom))
   )
@@
     (effects (font (size 1.27 1.27)) (justify left))
   )
-  (hierarchical_label "~CE" (shape input) (at 233.68 71.12 0)
-    (effects (font (size 1.27 1.27)) (justify left))
-  )

Commit message: Uploaded firmware v2.0.2
Connections:
- net R~W renamed R~{W}
- net ~CIA renamed ~{CIA}
- net ~CIAEXT renamed ~{CIAEXT}
- net ~OE renamed ~{OE}
- net ~PHI2 renamed ~{PHI2}
- net ~VIA renamed ~{VIA}
- net ~WE renamed ~{WE}
