File: kicad/peripherals.kicad_sch (KiCad schematic)
At the start: 7 parts, among them P2 5k, U1 6526, U11 74ACT245, U2 W65C22SxP

Commit message: v2.0
Production ready
Other:
- company: (none) -> Daniel Molina García
- title: (none) -> SBC6526 - Peripherals
Changed lines of the file:
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@@
 (kicad_sch (version 20201015) (generator eeschema)
   (paper "A4")
+  (title_block
+    (title "SBC6526 - Peripherals")
+    (date "2021-10-01")
+    (rev "2.0")
+    (company "Daniel Molina García")
+  )
   (junction (at 38.1 57.15) (diameter 1.016) (color 0 0 0 0))
   (junction (at 39.37 62.23) (diameter 1.016) (color 0 0 0 0))
@@
   (junction (at 162.56 128.27) (diameter 1.016) (color 0 0 0 0))
   (junction (at 243.84 163.83) (diameter 1.016) (color 0 0 0 0))
-  (no_connect (at 224.79 76.2))
+  (no_connect (at 224.79 96.52))
   (no_connect (at 224.79 106.68))
   (no_connect (at 224.79 78.74))
+  (no_connect (at 224.79 101.6))
+  (no_connect (at 224.79 76.2))
   (no_connect (at 224.79 109.22))
-  (no_connect (at 224.79 101.6))
-  (no_connect (at 224.79 96.52))
   (bus_entry (at 46.99 72.39) (size -2.54 2.54)
     (stroke (width 0.1524) (type solid) (color 0 0 0 0))
@@
     (effects (font (size 1.27 1.27)) (justify right bottom))
   )
-  (global_label "D[0..7]" (shape bidirectional) (at 185.42 130.81 0)    (property "Intersheet References" "${INTERSHEET_REFS}" (id 0) (at 195.949 130.7306 0)
-      (effects (font (size 1.27 1.27)) (justify left) hide)
-    )
-    (effects (font (size 1.27 1.27)) (justify left))
-  )
   (hierarchical_label "TODENABLE" (shape output) (at 35.56 22.86 180)

Commit message: Fixes
* Minor fixes to routing
* Right VCC hole was slightly offset. Fixed
* Removed /CE from arduino to RAM. As RAMCE pulses with PHI, it's not necessary, and we leave /CE tied to GND.
* Fixed RAM footprint, as it was too wide. Improved routing.
* Added current limiting resistor to LCD Contrast
Parts:
- added R20: 1k, Resistor_SMD:R_0805_2012Metric_Pad1.20x1.40mm_HandSolder, symbol Device:R
Connections:
- net GND: now also R20.2; no longer P2.1
- new net: P2.1, R20.1
Changed lines of the file:
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@@
   (junction (at 161.29 130.81) (diameter 1.016) (color 0 0 0 0))
   (junction (at 162.56 128.27) (diameter 1.016) (color 0 0 0 0))
-  (junction (at 243.84 163.83) (diameter 1.016) (color 0 0 0 0))
+  (no_connect (at 224.79 78.74))
+  (no_connect (at 224.79 76.2))
+  (no_connect (at 224.79 96.52))
+  (no_connect (at 224.79 109.22))
+  (no_connect (at 224.79 101.6))
   (no_connect (at 224.79 106.68))
-  (no_connect (at 224.79 76.2))
-  (no_connect (at 224.79 109.22))
-  (no_connect (at 224.79 96.52))
-  (no_connect (at 224.79 78.74))
-  (no_connect (at 224.79 101.6))
   (bus_entry (at 46.99 72.39) (size -2.54 2.54)
     (stroke (width 0.1524) (type solid) (color 0 0 0 0))
@@
     (stroke (width 0) (type solid) (color 0 0 0 0))
   )
-  (wire (pts (xy 279.4 29.21) (xy 279.4 33.02))
-    (stroke (width 0) (type solid) (color 0 0 0 0))
-  )
   (wire (pts (xy 281.94 60.96) (xy 281.94 63.5))
     (stroke (width 0) (type solid) (color 0 0 0 0))
@@
   )
   (bus (pts (xy 243.84 163.83) (xy 223.52 163.83))
-    (stroke (width 0) (type solid) (color 0 0 0 0))
-  )
-  (bus (pts (xy 267.97 163.83) (xy 243.84 163.83))
     (stroke (width 0) (type solid) (color 0 0 0 0))
   )
@@
     )
   )
-  (symbol (lib_id "power:GND") (at 279.4 33.02 0) (unit 1)
-    (in_bom yes) (on_board yes)
-    (property "Reference" "#PWR0121" (id 0) (at 279.4 39.37 0)
-      (effects (font (size 1.27 1.27)) hide)
-    )
-    (property "Value" "GND" (id 1) (at 279.527 37.4142 0))
-    (property "Footprint" "" (id 2) (at 279.4 33.02 0)
-      (effects (font (size 1.27 1.27)) hide)
-    )
-    (property "Datasheet" "" (id 3) (at 279.4 33.02 0)
+  (symbol (lib_id "power:GND") (at 279.4 36.83 0) (unit 1)
+    (in_bom yes) (on_board yes)
+    (property "Reference" "#PWR0121" (id 0) (at 279.4 43.18 0)
+      (effects (font (size 1.27 1.27)) hide)
+    )
+    (property "Value" "GND" (id 1) (at 279.527 41.2242 0))
+    (property "Footprint" "" (id 2) (at 279.4 36.83 0)
+      (effects (font (size 1.27 1.27)) hide)
+    )
+    (property "Datasheet" "" (id 3) (at 279.4 36.83 0)
       (effects (font (size 1.27 1.27)) hide)
     )
@@
     )
     (property "Datasheet" "~" (id 3) (at 278.13 54.61 0)
+      (effects (font (size 1.27 1.27)) hide)
+    )
+  )
+  (symbol (lib_id "Device:R") (at 279.4 33.02 0) (unit 1)
+    (in_bom yes) (on_board yes)
+    (property "Reference" "R20" (id 0) (at 281.178 31.8516 0)
+      (effects (font (size 1.27 1.27)) (justify left))
+    )
+    (property "Value" "1k" (id 1) (at 281.178 34.163 0)
+      (effects (font (size 1.27 1.27)) (justify left))
+    )
+    (property "Footprint" "Resistor_SMD:R_0805_2012Metric_Pad1.20x1.40mm_HandSolder" (id 2) (at 277.622 33.02 90)
+      (effects (font (size 1.27 1.27)) hide)
+    )
+    (property "Datasheet" "~" (id 3) (at 279.4 33.02 0)
       (effects (font (size 1.27 1.27)) hide)
     )
@@
     (in_bom yes) (on_board yes)
     (property "Reference" "LCD1" (id 0) (at 259.08 36.83 0))
-    (property "Value" "NHD-0420H1Z" (id 1) (at 270.51 36.83 0)
+    (property "Value" "NHD-0420H1Z" (id 1) (at 257.81 50.8 0)
       (effects (font (size 1.27 1.27)) (justify left))
     )

Commit message: Uploaded firmware v2.0.2
Connections:
- net R~W renamed R~{W}
- net ~CIA renamed ~{CIA}
- net ~CIAEXT renamed ~{CIAEXT}
- net ~CIARES renamed ~{CIARES}
- net ~EXTFLAG renamed ~{EXTFLAG}
- net ~EXTPC renamed ~{EXTPC}
- net ~IRQ renamed ~{IRQ}
- net ~RES renamed ~{RES}
- net ~VIA renamed ~{VIA}
- net ~VIAIRQ renamed ~{VIAIRQ}

Commit message: PullUps con SERCLOCK and SERDAT
Parts:
- added R21, R22: 3k3, Resistor_SMD:R_0805_2012Metric_Pad1.20x1.40mm_HandSolder, symbol Device:R
Connections:
- net SERCLK: now also R21.2
- net SERDAT: now also R22.2
- net VCC: now also R21.1, R22.1
Changed lines of the file:
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@@
   (junction (at 46.99 121.92) (diameter 1.016) (color 0 0 0 0)
   )
+  (junction (at 175.26 137.16) (diameter 0) (color 0 0 0 0)
+  )
   (junction (at 156.21 121.92) (diameter 1.016) (color 0 0 0 0)
   )
@@
   (junction (at 38.1 57.15) (diameter 1.016) (color 0 0 0 0)
   )
+  (junction (at 165.1 134.62) (diameter 0) (color 0 0 0 0)
+  )
   (junction (at 156.21 33.02) (diameter 1.016) (color 0 0 0 0)
   )
@@
   )
   (junction (at 41.91 67.31) (diameter 1.016) (color 0 0 0 0)
+  )
+  (junction (at 163.83 137.16) (diameter 0) (color 0 0 0 0)
   )
   (no_connect (at 224.79 109.22))
@@
     (stroke (width 0) (type solid) (color 0 0 0 0))
   )
+  (wire (pts (xy 179.07 137.16) (xy 179.07 139.7))
+    (stroke (width 0) (type default) (color 0 0 0 0))
+  )
   (wire (pts (xy 128.27 93.98) (xy 138.43 93.98))
     (stroke (width 0) (type solid) (color 0 0 0 0))
@@
     (stroke (width 0) (type solid) (color 0 0 0 0))
   )
+  (wire (pts (xy 163.83 152.4) (xy 179.07 152.4))
+    (stroke (width 0) (type default) (color 0 0 0 0))
+  )
   (wire (pts (xy 88.9 59.69) (xy 119.38 59.69))
     (stroke (width 0) (type solid) (color 0 0 0 0))
@@
     (stroke (width 0) (type solid) (color 0 0 0 0))
   )
+  (wire (pts (xy 179.07 147.32) (xy 179.07 152.4))
+    (stroke (width 0) (type default) (color 0 0 0 0))
+  )
   (bus (pts (xy 125.73 104.14) (xy 125.73 106.68))
     (stroke (width 0) (type solid) (color 0 0 0 0))
@@
     (stroke (width 0) (type solid) (color 0 0 0 0))
   )
+  (wire (pts (xy 165.1 134.62) (xy 165.1 151.13))
+    (stroke (width 0) (type default) (color 0 0 0 0))
+  )
   (bus (pts (xy 185.42 111.76) (xy 185.42 130.81))
     (stroke (width 0) (type solid) (color 0 0 0 0))
@@
     (stroke (width 0) (type solid) (color 0 0 0 0))
   )
+  (wire (pts (xy 175.26 137.16) (xy 179.07 137.16))
+    (stroke (width 0) (type default) (color 0 0 0 0))
+  )
   (bus (pts (xy 243.84 91.44) (xy 243.84 93.98))
     (stroke (width 0) (type solid) (color 0 0 0 0))
@@
     (stroke (width 0) (type solid) (color 0 0 0 0))
   )
+  (wire (pts (xy 165.1 151.13) (xy 172.72 151.13))
+    (stroke (width 0) (type default) (color 0 0 0 0))
+  )
   (wire (pts (xy 265.43 76.2) (xy 265.43 77.47))
     (stroke (width 0) (type solid) (color 0 0 0 0))
@@
     (stroke (width 0) (type solid) (color 0 0 0 0))
   )
+  (wire (pts (xy 172.72 139.7) (xy 172.72 137.16))
+    (stroke (width 0) (type default) (color 0 0 0 0))
+  )
   (wire (pts (xy 46.99 121.92) (xy 156.21 121.92))
     (stroke (width 0) (type solid) (color 0 0 0 0))
@@
     (stroke (width 0) (type solid) (color 0 0 0 0))
   )
+  (wire (pts (xy 172.72 137.16) (xy 175.26 137.16))
+    (stroke (width 0) (type default) (color 0 0 0 0))
+  )
   (wire (pts (xy 194.31 104.14) (xy 187.96 104.14))
     (stroke (width 0) (type solid) (color 0 0 0 0))
@@
     (stroke (width 0) (type solid) (color 0 0 0 0))
   )
+  (wire (pts (xy 172.72 147.32) (xy 172.72 151.13))
+    (stroke (width 0) (type default) (color 0 0 0 0))
+  )
   (wire (pts (xy 224.79 60.96) (xy 236.22 60.96))
     (stroke (width 0) (type solid) (color 0 0 0 0))
@@
   (wire (pts (xy 124.46 111.76) (xy 124.46 35.56))
     (stroke (width 0) (type solid) (color 0 0 0 0))
+  )
+  (wire (pts (xy 163.83 137.16) (xy 163.83 152.4))
+    (stroke (width 0) (type default) (color 0 0 0 0))
   )
   (wire (pts (xy 39.37 62.23) (xy 35.56 62.23))
@@
     (pin "1")
   )
+  (symbol (lib_id "power:VCC") (at 175.26 137.16 0) (unit 1)
+    (in_bom yes) (on_board yes)
+    (property "Reference" "#PWR03" (id 0) (at 175.26 140.97 0)
+      (effects (font (size 1.27 1.27)) hide)
+    )
+    (property "Value" "VCC" (id 1) (at 175.641 132.7658 0))
+    (property "Footprint" "" (id 2) (at 175.26 137.16 0)
+      (effects (font (size 1.27 1.27)) hide)
+    )
+    (property "Datasheet" "" (id 3) (at 175.26 137.16 0)
+      (effects (font (size 1.27 1.27)) hide)
+    )
+    (pin "1")
+  )
   (symbol (lib_id "Device:R") (at 279.4 33.02 0) (unit 1)
     (in_bom yes) (on_board yes)
@@
       (effects (font (size 1.27 1.27)) hide)
     )
+    (pin "1")
+    (pin "2")
+  )
+  (symbol (lib_id "Device:R") (at 179.07 143.51 0) (mirror y) (unit 1)
+    (in_bom yes) (on_board yes)
+    (property "Reference" "R22" (id 0) (at 177.292 142.3416 0)
+      (effects (font (size 1.27 1.27)) (justify left))
+    )
+    (property "Value" "3k3" (id 1) (at 177.292 144.653 0)
+      (effects (font (size 1.27 1.27)) (justify left))
+    )
+    (property "Footprint" "Resistor_SMD:R_0805_2012Metric_Pad1.20x1.40mm_HandSolder" (id 2) (at 180.848 143.51 90)
+      (effects (font (size 1.27 1.27)) hide)
+    )
+    (property "Datasheet" "~" (id 3) (at 179.07 143.51 0)
+      (effects (font (size 1.27 1.27)) hide)
+    )
+    (pin "1")
+    (pin "2")
+  )
+  (symbol (lib_id "Device:R") (at 172.72 143.51 0) (unit 1)
+    (in_bom yes) (on_board yes)
+    (property "Reference" "R21" (id 0) (at 174.498 142.3416 0)
+      (effects (font (size 1.27 1.27)) (justify left))
+    )
+    (property "Value" "3k3" (id 1) (at 174.498 144.653 0)
+      (effects (font (size 1.27 1.27)) (justify left))
+    )
+    (property "Footprint" "Resistor_SMD:R_0805_2012Metric_Pad1.20x1.40mm_HandSolder" (id 2) (at 170.942 143.51 90)
+      (effects (font (size 1.27 1.27)) hide)
+    )
+    (property "Datasheet" "~" (id 3) (at 172.72 143.51 0)
+      (effects (font (size 1.27 1.27)) hide)
+    )
