File: kicad/power.kicad_sch (KiCad schematic)
At the start: 14 parts, among them U7 74AC74, U8 74AC14, U9 74AC139

Commit message: v2.0
Production ready
Other:
- company: (none) -> Daniel Molina García
- title: (none) -> SBC6526 - Power
Changed lines of the file:
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@@
 (kicad_sch (version 20201015) (generator eeschema)
   (paper "A4")
+  (title_block
+    (title "SBC6526 - Power")
+    (date "2021-10-01")
+    (rev "2.0")
+    (company "Daniel Molina García")
+  )
   (junction (at 48.26 43.18) (diameter 1.016) (color 0 0 0 0))
   (junction (at 48.26 53.34) (diameter 1.016) (color 0 0 0 0))
@@
   (no_connect (at 63.5 181.61))
   (no_connect (at 64.77 148.59))
+  (no_connect (at 63.5 166.37))
+  (no_connect (at 63.5 176.53))
   (no_connect (at 63.5 157.48))
-  (no_connect (at 63.5 176.53))
-  (no_connect (at 63.5 166.37))
   (wire (pts (xy 48.26 33.02) (xy 48.26 43.18))
     (stroke (width 0) (type solid) (color 0 0 0 0))
