File: kicad/reset.kicad_sch (KiCad schematic)
At the start: 6 parts, among them SW5 RESET, U8 74AC14

Commit message: v2.0
Production ready
Other:
- company: (none) -> Daniel Molina García
- title: (none) -> SBC6526 - Reset
Changed lines of the file:
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@@
 (kicad_sch (version 20201015) (generator eeschema)
   (paper "A4")
+  (title_block
+    (title "SBC6526 - Reset")
+    (date "2021-10-01")
+    (rev "2.0")
+    (company "Daniel Molina García")
+  )
   (junction (at 102.87 99.06) (diameter 1.016) (color 0 0 0 0))
   (junction (at 140.97 99.06) (diameter 1.016) (color 0 0 0 0))

Commit message: Uploaded firmware v2.0.2
Connections:
- net ~RES renamed ~{RES}
Changed lines of the file:
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@@
-(kicad_sch (version 20201015) (generator eeschema)
+(kicad_sch (version 20211123) (generator eeschema)
   (paper "A4")
   (title_block
@@
     (company "Daniel Molina García")
   )
-  (junction (at 102.87 99.06) (diameter 1.016) (color 0 0 0 0))
-  (junction (at 140.97 99.06) (diameter 1.016) (color 0 0 0 0))
-  (junction (at 165.1 99.06) (diameter 1.016) (color 0 0 0 0))
-  (wire (pts (xy 102.87 68.58) (xy 102.87 74.93))
+  (junction (at 102.87 99.06) (diameter 1.016) (color 0 0 0 0)
+  )
+  (junction (at 140.97 99.06) (diameter 1.016) (color 0 0 0 0)
+  )
+  (junction (at 165.1 99.06) (diameter 1.016) (color 0 0 0 0)
+  )
+  (wire (pts (xy 165.1 99.06) (xy 165.1 68.58))
+    (stroke (width 0) (type solid) (color 0 0 0 0))
+  )
+  (wire (pts (xy 165.1 68.58) (xy 158.75 68.58))
+    (stroke (width 0) (type solid) (color 0 0 0 0))
+  )
+  (wire (pts (xy 140.97 83.82) (xy 140.97 99.06))
+    (stroke (width 0) (type solid) (color 0 0 0 0))
+  )
+  (wire (pts (xy 165.1 99.06) (xy 171.45 99.06))
+    (stroke (width 0) (type solid) (color 0 0 0 0))
+  )
+  (wire (pts (xy 133.35 99.06) (xy 140.97 99.06))
     (stroke (width 0) (type solid) (color 0 0 0 0))
   )
@@
     (stroke (width 0) (type solid) (color 0 0 0 0))
   )
+  (wire (pts (xy 140.97 76.2) (xy 140.97 68.58))
+    (stroke (width 0) (type solid) (color 0 0 0 0))
+  )
   (wire (pts (xy 102.87 99.06) (xy 102.87 114.3))
+    (stroke (width 0) (type solid) (color 0 0 0 0))
+  )
+  (wire (pts (xy 157.48 99.06) (xy 165.1 99.06))
+    (stroke (width 0) (type solid) (color 0 0 0 0))
+  )
+  (wire (pts (xy 186.69 99.06) (xy 201.93 99.06))
     (stroke (width 0) (type solid) (color 0 0 0 0))
   )
@@
     (stroke (width 0) (type solid) (color 0 0 0 0))
   )
-  (wire (pts (xy 125.73 99.06) (xy 102.87 99.06))
-    (stroke (width 0) (type solid) (color 0 0 0 0))
-  )
-  (wire (pts (xy 133.35 99.06) (xy 140.97 99.06))
-    (stroke (width 0) (type solid) (color 0 0 0 0))
-  )
-  (wire (pts (xy 140.97 76.2) (xy 140.97 68.58))
-    (stroke (width 0) (type solid) (color 0 0 0 0))
-  )
-  (wire (pts (xy 140.97 83.82) (xy 140.97 99.06))
-    (stroke (width 0) (type solid) (color 0 0 0 0))
-  )
   (wire (pts (xy 140.97 99.06) (xy 149.86 99.06))
     (stroke (width 0) (type solid) (color 0 0 0 0))
   )
-  (wire (pts (xy 157.48 99.06) (xy 165.1 99.06))
+  (wire (pts (xy 102.87 68.58) (xy 102.87 74.93))
     (stroke (width 0) (type solid) (color 0 0 0 0))
   )
-  (wire (pts (xy 165.1 68.58) (xy 158.75 68.58))
-    (stroke (width 0) (type solid) (color 0 0 0 0))
-  )
-  (wire (pts (xy 165.1 99.06) (xy 165.1 68.58))
-    (stroke (width 0) (type solid) (color 0 0 0 0))
-  )
-  (wire (pts (xy 165.1 99.06) (xy 171.45 99.06))
-    (stroke (width 0) (type solid) (color 0 0 0 0))
-  )
-  (wire (pts (xy 186.69 99.06) (xy 201.93 99.06))
+  (wire (pts (xy 125.73 99.06) (xy 102.87 99.06))
     (stroke (width 0) (type solid) (color 0 0 0 0))
   )
@@
     (effects (font (size 1.27 1.27)) (justify right))
   )
-  (hierarchical_label "~RES" (shape output) (at 201.93 99.06 0)
+  (hierarchical_label "~{RES}" (shape output) (at 201.93 99.06 0)
     (effects (font (size 1.27 1.27)) (justify left))
   )
-  (symbol (lib_id "power:VCC") (at 102.87 68.58 0) (unit 1)
+  (symbol (lib_id "74xx:74LS14") (at 179.07 99.06 0) (unit 6)
     (in_bom yes) (on_board yes)
-    (property "Reference" "#PWR0113" (id 0) (at 102.87 72.39 0)
+    (property "Reference" "U8" (id 0) (at 179.07 91.0082 0))
+    (property "Value" "74AC14" (id 1) (at 179.07 93.3196 0))
+    (property "Footprint" "Package_SO:SOIC-14_3.9x8.7mm_P1.27mm" (id 2) (at 179.07 99.06 0)
       (effects (font (size 1.27 1.27)) hide)
     )
-    (property "Value" "VCC" (id 1) (at 103.251 64.1858 0))
-    (property "Footprint" "" (id 2) (at 102.87 68.58 0)
+    (property "Datasheet" "http://www.ti.com/lit/gpn/sn74LS14" (id 3) (at 179.07 99.06 0)
       (effects (font (size 1.27 1.27)) hide)
     )
-    (property "Datasheet" "" (id 3) (at 102.87 68.58 0)
-      (effects (font (size 1.27 1.27)) hide)
-    )
-  )
-  (symbol (lib_id "power:VCC") (at 140.97 68.58 0) (unit 1)
-    (in_bom yes) (on_board yes)
-    (property "Reference" "#PWR0114" (id 0) (at 140.97 72.39 0)
-      (effects (font (size 1.27 1.27)) hide)
-    )
-    (property "Value" "VCC" (id 1) (at 141.351 64.1858 0))
-    (property "Footprint" "" (id 2) (at 140.97 68.58 0)
-      (effects (font (size 1.27 1.27)) hide)
-    )
-    (property "Datasheet" "" (id 3) (at 140.97 68.58 0)
-      (effects (font (size 1.27 1.27)) hide)
-    )
-  )
-  (symbol (lib_id "power:GND") (at 102.87 129.54 0) (unit 1)
-    (in_bom yes) (on_board yes)
-    (property "Reference" "#PWR0115" (id 0) (at 102.87 135.89 0)
-      (effects (font (size 1.27 1.27)) hide)
-    )
-    (property "Value" "GND" (id 1) (at 102.997 133.9342 0))
-    (property "Footprint" "" (id 2) (at 102.87 129.54 0)
-      (effects (font (size 1.27 1.27)) hide)
-    )
-    (property "Datasheet" "" (id 3) (at 102.87 129.54 0)
-      (effects (font (size 1.27 1.27)) hide)
-    )
+    (pin "12")
+    (pin "13")
   )
   (symbol (lib_id "Device:R") (at 102.87 118.11 0) (unit 1)
@@
       (effects (font (size 1.27 1.27)) hide)
     )
+    (pin "1")
+    (pin "2")
+  )
+  (symbol (lib_id "Device:R") (at 153.67 99.06 270) (unit 1)
+    (in_bom yes) (on_board yes)
+    (property "Reference" "R12" (id 0) (at 153.67 93.8022 90))
+    (property "Value" "5,6k" (id 1) (at 153.67 96.1136 90))
+    (property "Footprint" "Resistor_SMD:R_0805_2012Metric_Pad1.20x1.40mm_HandSolder" (id 2) (at 153.67 97.282 90)
+      (effects (font (size 1.27 1.27)) hide)
+    )
+    (property "Datasheet" "~" (id 3) (at 153.67 99.06 0)
+      (effects (font (size 1.27 1.27)) hide)
+    )
+    (pin "1")
+    (pin "2")
   )
   (symbol (lib_id "Device:R") (at 129.54 99.06 270) (unit 1)
@@
       (effects (font (size 1.27 1.27)) hide)
     )
-  )
-  (symbol (lib_id "Device:R") (at 153.67 99.06 270) (unit 1)
-    (in_bom yes) (on_board yes)
-    (property "Reference" "R12" (id 0) (at 153.67 93.8022 90))
-    (property "Value" "5,6k" (id 1) (at 153.67 96.1136 90))
-    (property "Footprint" "Resistor_SMD:R_0805_2012Metric_Pad1.20x1.40mm_HandSolder" (id 2) (at 153.67 97.282 90)
-      (effects (font (size 1.27 1.27)) hide)
-    )
-    (property "Datasheet" "~" (id 3) (at 153.67 99.06 0)
-      (effects (font (size 1.27 1.27)) hide)
-    )
+    (pin "1")
+    (pin "2")
   )
   (symbol (lib_id "Device:C") (at 140.97 80.01 0) (unit 1)
@@
       (effects (font (size 1.27 1.27)) hide)
     )
+    (pin "1")
+    (pin "2")
   )
   (symbol (lib_id "Switch:SW_MEC_5G") (at 102.87 80.01 90) (unit 1)
@@
       (effects (font (size 1.27 1.27)) hide)
     )
+    (pin "1")
+    (pin "3")
+    (pin "2")
+    (pin "4")
   )
-  (symbol (lib_id "74xx:74LS14") (at 179.07 99.06 0) (unit 6)
+  (symbol (lib_id "power:VCC") (at 102.87 68.58 0) (unit 1)
     (in_bom yes) (on_board yes)
-    (property "Reference" "U8" (id 0) (at 179.07 91.0082 0))
-    (property "Value" "74AC14" (id 1) (at 179.07 93.3196 0))
-    (property "Footprint" "Package_SO:SOIC-14_3.9x8.7mm_P1.27mm" (id 2) (at 179.07 99.06 0)
+    (property "Reference" "#PWR0113" (id 0) (at 102.87 72.39 0)
       (effects (font (size 1.27 1.27)) hide)
     )
-    (property "Datasheet" "http://www.ti.com/lit/gpn/sn74LS14" (id 3) (at 179.07 99.06 0)
+    (property "Value" "VCC" (id 1) (at 103.251 64.1858 0))
+    (property "Footprint" "" (id 2) (at 102.87 68.58 0)
       (effects (font (size 1.27 1.27)) hide)
     )
+    (property "Datasheet" "" (id 3) (at 102.87 68.58 0)
+      (effects (font (size 1.27 1.27)) hide)
+    )
+    (pin "1")
+  )
+  (symbol (lib_id "power:VCC") (at 140.97 68.58 0) (unit 1)
+    (in_bom yes) (on_board yes)
+    (property "Reference" "#PWR0114" (id 0) (at 140.97 72.39 0)
+      (effects (font (size 1.27 1.27)) hide)
+    )
+    (property "Value" "VCC" (id 1) (at 141.351 64.1858 0))
+    (property "Footprint" "" (id 2) (at 140.97 68.58 0)
+      (effects (font (size 1.27 1.27)) hide)
+    )
+    (property "Datasheet" "" (id 3) (at 140.97 68.58 0)
+      (effects (font (size 1.27 1.27)) hide)
+    )
+    (pin "1")
+  )
+  (symbol (lib_id "power:GND") (at 102.87 129.54 0) (unit 1)
+    (in_bom yes) (on_board yes)
+    (property "Reference" "#PWR0115" (id 0) (at 102.87 135.89 0)
+      (effects (font (size 1.27 1.27)) hide)
+    )
+    (property "Value" "GND" (id 1) (at 102.997 133.9342 0))
+    (property "Footprint" "" (id 2) (at 102.87 129.54 0)
+      (effects (font (size 1.27 1.27)) hide)
+    )
+    (property "Datasheet" "" (id 3) (at 102.87 129.54 0)
+      (effects (font (size 1.27 1.27)) hide)
+    )
+    (pin "1")
   )
 )
